File: AutoFloppySwitcher.kicad_pcb (KiCad board)
At the start: 4 copper layers, 79.7 x 45.7 mm, 31 parts, among them J1 Wire Twist, J2 Berg Pwr in, J3 Power Passthrough, Q1 Q_NPN_CBE, Q2 BSS138, Q3 BSS138, Q4 Q_PNP_BEC, Q5 2N7002, Q6 BSS138, Q7 BSS138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

Commit message: update
Connections:
- net 555-Release renamed /555-Release
- net 555-Trigger renamed /555-Trigger
- net DSKCHG-Pulldown renamed /DSKCHG-Pulldown
Routing:
- net /RDATA: track 59.3 -> 60.1 mm
Other:
- board text added: "Floppy Drives"
Changed lines of the file:
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@@
       (outputformat 1)
       (mirror false)
-      (drillshape 1)
+      (drillshape 0)
       (scaleselection 1)
-      (outputdirectory "")
+      (outputdirectory "gerbers")
     )
   )
@@
   (net 9 "Net-(D1-Pad1)")
   (net 10 "GND")
-  (net 11 "555-Trigger")
+  (net 11 "/555-Trigger")
   (net 12 "Floppy-Drive-A")
   (net 13 "{slash}MOTEA-OUT")
@@
   (net 15 "Net-(Q4-Pad1)")
   (net 16 "+5V")
-  (net 17 "555-Release")
-  (net 18 "DSKCHG-Pulldown")
+  (net 17 "/555-Release")
+  (net 18 "/DSKCHG-Pulldown")
   (net 19 "{slash}DSKCHG")
   (net 20 "{slash}DRVSA-OUT")
@@
     (descr "Capacitor SMD 0805 (2012 Metric), square (rectangular) end terminal, IPC_7351 nominal, (Body size source: IPC-SM-782 page 76, https://www.pcb-3d.com/wordpress/wp-content/uploads/ipc-sm-782a_amendment_1_and_2.pdf, https://docs.google.com/spreadsheets/d/1BsfQQcO9C6DZCsRaXUlFlo91Tg2WpOkGARC1WS5S8t0/edit?usp=sharing), generated with kicad-footprint-generator")
     (tags "capacitor")
+    (property "JLCPCB" "C49678")
     (property "Sheetfile" "AutoFloppySwitcher.kicad_sch")
     (property "Sheetname" "")
@@
       (net 10 "GND") (pintype "passive") (solder_mask_margin 0.05))
     (pad "2" smd rect (at 0.95 0 180) (size 1 1.45) (layers "F.Cu" "F.Paste" "F.Mask")
-      (net 18 "DSKCHG-Pulldown") (pintype "passive") (solder_mask_margin 0.05))
+      (net 18 "/DSKCHG-Pulldown") (pintype "passive") (solder_mask_margin 0.05))
     (model "${KICAD6_3DMODEL_DIR}/Resistor_SMD.3dshapes/R_0805_2012Metric.wrl"
       (offset (xyz 0 0 0))
@@
     (fp_line (start -1 0.625) (end -1 -0.625) (layer "F.Fab") (width 0.1))
     (pad "1" smd rect (at -0.95 0) (size 1 1.45) (layers "F.Cu" "F.Paste" "F.Mask")
-      (net 11 "555-Trigger") (pintype "passive") (solder_mask_margin 0.05))
+      (net 11 "/555-Trigger") (pintype "passive") (solder_mask_margin 0.05))
     (pad "2" smd rect (at 0.95 0) (size 1 1.45) (layers "F.Cu" "F.Paste" "F.Mask")
       (net 16 "+5V") (pintype "passive") (solder_mask_margin 0.05))
@@
     (fp_line (start -0.88 -1) (end -0.43 -1.45) (layer "F.Fab") (width 0.1))
     (pad "1" smd rect (at -1.46 -0.95) (size 1.5 0.65) (layers "F.Cu" "F.Paste" "F.Mask")
-      (net 18 "DSKCHG-Pulldown") (pinfunction "G") (pintype "input") (solder_mask_margin 0.05))
+      (net 18 "/DSKCHG-Pulldown") (pinfunction "G") (pintype "input") (solder_mask_margin 0.05))
     (pad "2" smd rect (at -1.46 0.95) (size 1.5 0.65) (layers "F.Cu" "F.Paste" "F.Mask")
       (net 10 "GND") (pinfunction "S") (pintype "passive") (solder_mask_margin 0.05))
@@
       (net 10 "GND") (pintype "passive") (solder_mask_margin 0.05))
     (pad "2" smd rect (at 0.95 0 180) (size 1 1.45) (layers "F.Cu" "F.Paste" "F.Mask")
-      (net 17 "555-Release") (pintype "passive") (solder_mask_margin 0.05))
+      (net 17 "/555-Release") (pintype "passive") (solder_mask_margin 0.05))
     (model "${KICAD6_3DMODEL_DIR}/Resistor_SMD.3dshapes/R_0805_2012Metric.wrl"
       (offset (xyz 0 0 0))
@@
       (net 10 "GND") (pinfunction "GND") (pintype "power_in") (clearance 0.07))
     (pad "2" smd rect (at -2.475 -0.635 90) (size 1.95 0.6) (layers "F.Cu" "F.Paste" "F.Mask")
-      (net 11 "555-Trigger") (pinfunction "TR") (pintype "input") (clearance 0.07))
+      (net 11 "/555-Trigger") (pinfunction "TR") (pintype "input") (clearance 0.07))
     (pad "3" smd rect (at -2.475 0.635 90) (size 1.95 0.6) (layers "F.Cu" "F.Paste" "F.Mask")
-      (net 18 "DSKCHG-Pulldown") (pinfunction "Q") (pintype "output") (clearance 0.07))
+      (net 18 "/DSKCHG-Pulldown") (pinfunction "Q") (pintype "output") (clearance 0.07))
     (pad "4" smd rect (at -2.475 1.905 90) (size 1.95 0.6) (layers "F.Cu" "F.Paste" "F.Mask")
       (net 22 "Net-(R3-Pad2)") (pinfunction "R") (pintype "input") (clearance 0.07))
@@
       (net 24 "unconnected-(U1-Pad5)") (pinfunction "CV") (pintype "input+no_connect") (clearance 0.07))
     (pad "6" smd rect (at 2.475 0.635 90) (size 1.95 0.6) (layers "F.Cu" "F.Paste" "F.Mask")
-      (net 17 "555-Release") (pinfunction "THR") (pintype "input") (clearance 0.07))
+      (net 17 "/555-Release") (pinfunction "THR") (pintype "input") (clearance 0.07))
     (pad "7" smd rect (at 2.475 -0.635 90) (size 1.95 0.6) (layers "F.Cu" "F.Paste" "F.Mask")
       (net 25 "unconnected-(U1-Pad7)") (pinfunction "DIS") (pintype "input+no_connect") (clearance 0.07))
@@
       (net 10 "GND") (pinfunction "E") (pintype "passive") (solder_mask_margin 0.05))
     (pad "3" smd rect (at 1.46 0) (size 1.5 0.65) (layers "F.Cu" "F.Paste" "F.Mask")
-      (net 11 "555-Trigger") (pinfunction "C") (pintype "passive") (solder_mask_margin 0.05))
+      (net 11 "/555-Trigger") (pinfunction "C") (pintype "passive") (solder_mask_margin 0.05))
     (model "${KICAD6_3DMODEL_DIR}/Package_TO_SOT_SMD.3dshapes/TSOT-23.wrl"
       (offset (xyz 0 0 0))
@@
       (net 16 "+5V") (pinfunction "E") (pintype "passive") (solder_mask_margin 0.05))
     (pad "3" smd rect (at 1.46 0) (size 1.5 0.65) (layers "F.Cu" "F.Paste" "F.Mask")
-      (net 17 "555-Release") (pinfunction "C") (pintype "passive") (solder_mask_margin 0.05))
+      (net 17 "/555-Release") (pinfunction "C") (pintype "passive") (solder_mask_margin 0.05))
     (model "${KICAD6_3DMODEL_DIR}/Package_TO_SOT_SMD.3dshapes/TSOT-23.wrl"
       (offset (xyz 0 0 0))
@@
   (gr_line (start 74.997 56.8425) (end 73.981 57.8585) (layer "Edge.Cuts") (width 0.1))
   (gr_line (start 83.058 56.8425) (end 150.67 56.8425) (layer "Edge.Cuts") (width 0.1))
+  (gr_text "Floppy Drives" (at 130.302 92.456 90) (layer "F.SilkS")
+    (effects (font (size 1.8 1.8) (thickness 0.3)))
+  )
   (gr_text "Host" (at 86.487 69.215 90) (layer "F.SilkS")
     (effects (font (size 2 2) (thickness 0.3)))
@@
   (segment (start 110.522 78.994) (end 112.044 78.994) (width 0.6) (layer "F.Cu") (net 16))
   (segment (start 125.479 78.867) (end 125.54 78.928) (width 0.3) (layer "F.Cu") (net 16))
+  (segment (start 128.27 97.68) (end 127.95 98) (width 0.3) (layer "F.Cu") (net 16))
   (segment (start 112.044 78.994) (end 112.05 79) (width 0.6) (layer "F.Cu") (net 16))
   (segment (start 118.5992 80.3168) (end 118.587 80.329) (width 0.6) (layer "F.Cu") (net 16))
+  (segment (start 128.27 96.266) (end 128.27 97.68) (width 0.3) (layer "F.Cu") (net 16))
   (segment (start 110.522 82.8) (end 112.05 82.8) (width 0.6) (layer "F.Cu") (net 16))
   (segment (start 123.698 78.867) (end 125.479 78.867) (width 0.3) (layer "F.Cu") (net 16))
-  (segment (start 129.496 98) (end 129.54 98.044) (width 0.3) (layer "F.Cu") (net 16))
-  (segment (start 127.95 98) (end 129.496 98) (width 0.3) (layer "F.Cu") (net 16))
   (segment (start 110.522 86.6) (end 112.05 86.6) (width 0.6) (layer "F.Cu") (net 16))
   (via (at 123.698 78.867) (size 0.8) (drill 0.4) (layers "F.Cu" "B.Cu") (free) (net 16))
   (via (at 118.5992 78.359) (size 0.8) (drill 0.4) (layers "F.Cu" "B.Cu") (free) (net 16))
   (via (at 110.522 82.8) (size 0.8) (drill 0.4) (layers "F.Cu" "B.Cu") (free) (net 16))
-  (via (at 129.54 98.044) (size 0.8) (drill 0.4) (layers "F.Cu" "B.Cu") (free) (net 16))
+  (via (at 128.27 96.266) (size 0.8) (drill 0.4) (layers "F.Cu" "B.Cu") (free) (net 16))
   (via (at 110.522 86.6) (size 0.8) (drill 0.4) (layers "F.Cu" "B.Cu") (free) (net 16))
   (via (at 110.522 90.424) (size 0.8) (drill 0.4) (layers "F.Cu" "B.Cu") (free) (net 16))
@@
   (segment (start 85.725 94.996) (end 78.994 94.996) (width 0.3) (layer "F.Cu") (net 34))
   (segment (start 94.356 94.991) (end 93.147 96.2) (width 0.3) (layer "F.Cu") (net 34))
+  (segment (start 127 95.25) (end 126.05 96.2) (width 0.3) (layer "In2.Cu") (net 34))
   (segment (start 94.356 94.996) (end 95.56 96.2) (width 0.3) (layer "In2.Cu") (net 34))
+  (segment (start 130.495 96.2) (end 129.545 95.25) (width 0.3) (layer "In2.Cu") (net 34))
   (segment (start 135.102 96.2) (end 136.311 94.991) (width 0.3) (layer "In2.Cu") (net 34))
-  (segment (start 95.56 96.2) (end 135.102 96.2) (width 0.3) (layer "In2.Cu") (net 34))
+  (segment (start 129.545 95.25) (end 127 95.25) (width 0.3) (layer "In2.Cu") (net 34))
+  (segment (start 130.495 96.2) (end 135.102 96.2) (width 0.3) (layer "In2.Cu") (net 34))
+  (segment (start 95.56 96.2) (end 126.05 96.2) (width 0.3) (layer "In2.Cu") (net 34))
   (segment (start 86.939 98.75) (end 85.725 97.536) (width 0.3) (layer "F.Cu") (net 35))
   (segment (start 93.137 98.75) (end 86.939 98.75) (width 0.3) (layer "F.Cu") (net 35))
