File: AutoFloppySwitcher.kicad_sch (KiCad schematic)
At the start: 28 parts, among them J1 Wire Twist, J2 Berg Pwr in, J3 Power Passthrough, Q1 Q_NPN_CBE, Q2 BSS138, Q3 BSS138, Q4 Q_PNP_BEC, Q5 2N7002, Q6 BSS138, Q7 BSS138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

Commit message: update
Parts:
- C1: JLCPCB (none) -> C49678
Changed lines of the file:
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@@
   (junction (at 382.27 186.69) (diameter 0) (color 0 0 0 0)
   )
-  (junction (at 212.09 218.44) (diameter 0) (color 0 0 0 0)
-  )
   (junction (at 382.27 209.55) (diameter 0) (color 0 0 0 0)
   )
@@
   (junction (at 90.17 138.43) (diameter 0) (color 0 0 0 0)
   )
-  (junction (at 212.09 165.1) (diameter 0) (color 0 0 0 0)
-  )
   (junction (at 106.68 77.47) (diameter 0) (color 0 0 0 0)
   )
@@
   )
   (junction (at 246.38 58.42) (diameter 0) (color 0 0 0 0)
-  )
-  (junction (at 109.22 195.58) (diameter 0) (color 0 0 0 0)
   )
   (junction (at 382.27 66.04) (diameter 0) (color 0 0 0 0)
@@
     (stroke (width 0) (type default) (color 0 0 0 0))
   )
-  (wire (pts (xy 212.09 165.1) (xy 241.3 165.1))
-    (stroke (width 0) (type default) (color 0 0 0 0))
-  )
   (wire (pts (xy 356.87 58.42) (xy 354.33 58.42))
     (stroke (width 0) (type default) (color 0 0 0 0))
@@
     (stroke (width 0) (type default) (color 0 0 0 0))
   )
-  (wire (pts (xy 111.76 190.5) (xy 109.22 190.5))
-    (stroke (width 0) (type default) (color 0 0 0 0))
-  )
   (wire (pts (xy 356.87 113.03) (xy 354.33 113.03))
     (stroke (width 0) (type default) (color 0 0 0 0))
@@
     (stroke (width 0) (type default) (color 0 0 0 0))
   )
-  (wire (pts (xy 194.31 165.1) (xy 212.09 165.1))
+  (wire (pts (xy 194.31 165.1) (xy 241.3 165.1))
     (stroke (width 0) (type default) (color 0 0 0 0))
   )
@@
     (stroke (width 0) (type default) (color 0 0 0 0))
   )
-  (wire (pts (xy 212.09 168.91) (xy 212.09 165.1))
-    (stroke (width 0) (type default) (color 0 0 0 0))
-  )
   (polyline (pts (xy 209.55 147.32) (xy 209.55 226.06))
     (stroke (width 0) (type default) (color 0 0 0 0))
@@
     (stroke (width 0) (type default) (color 0 0 0 0))
   )
-  (wire (pts (xy 109.22 190.5) (xy 109.22 195.58))
-    (stroke (width 0) (type default) (color 0 0 0 0))
-  )
   (wire (pts (xy 356.87 118.11) (xy 354.33 118.11))
     (stroke (width 0) (type default) (color 0 0 0 0))
@@
     (stroke (width 0) (type default) (color 0 0 0 0))
   )
-  (wire (pts (xy 194.31 218.44) (xy 212.09 218.44))
+  (wire (pts (xy 194.31 218.44) (xy 240.03 218.44))
     (stroke (width 0) (type default) (color 0 0 0 0))
   )
@@
     (stroke (width 0) (type default) (color 0 0 0 0))
   )
-  (wire (pts (xy 212.09 222.25) (xy 212.09 218.44))
-    (stroke (width 0) (type default) (color 0 0 0 0))
-  )
   (polyline (pts (xy 138.43 54.61) (xy 138.43 101.6))
     (stroke (width 0) (type default) (color 0 0 0 0))
@@
     (stroke (width 0) (type default) (color 0 0 0 0))
   )
-  (wire (pts (xy 214.63 168.91) (xy 212.09 168.91))
-    (stroke (width 0) (type default) (color 0 0 0 0))
-  )
   (wire (pts (xy 252.73 156.21) (xy 252.73 160.02))
     (stroke (width 0) (type default) (color 0 0 0 0))
@@
     (stroke (width 0) (type default) (color 0 0 0 0))
   )
-  (wire (pts (xy 214.63 222.25) (xy 212.09 222.25))
-    (stroke (width 0) (type default) (color 0 0 0 0))
-  )
   (wire (pts (xy 356.87 86.36) (xy 354.33 86.36))
     (stroke (width 0) (type default) (color 0 0 0 0))
@@
   )
   (wire (pts (xy 356.87 151.13) (xy 354.33 151.13))
-    (stroke (width 0) (type default) (color 0 0 0 0))
-  )
-  (wire (pts (xy 212.09 218.44) (xy 240.03 218.44))
     (stroke (width 0) (type default) (color 0 0 0 0))
   )
@@
   )
   (text "Floppy drive switch" (at 157.48 59.69 0)
+    (effects (font (size 1.27 1.27)) (justify left bottom))
+  )
+  (label "555-Release" (at 212.09 218.44 0)
+    (effects (font (size 1.27 1.27)) (justify left bottom))
+  )
+  (label "555-Trigger" (at 109.22 195.58 0)
+    (effects (font (size 1.27 1.27)) (justify left bottom))
+  )
+  (label "DSKCHG-Pulldown" (at 212.09 165.1 0)
     (effects (font (size 1.27 1.27)) (justify left bottom))
   )
@@
     )
   )
-  (global_label "DSKCHG-Pulldown" (shape input) (at 214.63 168.91 0) (fields_autoplaced)
-    (effects (font (size 1.27 1.27)) (justify left))
-    (property "Intersheet References" "${INTERSHEET_REFS}" (id 0) (at 234.7626 168.8306 0)
-      (effects (font (size 1.27 1.27)) (justify left) hide)
-    )
-  )
   (global_label "{slash}WPT" (shape input) (at 354.33 81.28 180) (fields_autoplaced)
     (effects (font (size 1.27 1.27)) (justify right))
@@
     (property "Intersheet References" "${INTERSHEET_REFS}" (id 0) (at 345.1436 151.2094 0)
       (effects (font (size 1.27 1.27)) (justify right) hide)
-    )
-  )
-  (global_label "555-Release" (shape input) (at 214.63 222.25 0) (fields_autoplaced)
-    (effects (font (size 1.27 1.27)) (justify left))
-    (property "Intersheet References" "${INTERSHEET_REFS}" (id 0) (at 229.6221 222.3294 0)
-      (effects (font (size 1.27 1.27)) (justify left) hide)
     )
   )
@@
     (effects (font (size 1.27 1.27)) (justify left))
     (property "Intersheet References" "${INTERSHEET_REFS}" (id 0) (at 264.0936 88.8206 0)
-      (effects (font (size 1.27 1.27)) (justify left) hide)
-    )
-  )
-  (global_label "555-Trigger" (shape input) (at 111.76 190.5 0) (fields_autoplaced)
-    (effects (font (size 1.27 1.27)) (justify left))
-    (property "Intersheet References" "${INTERSHEET_REFS}" (id 0) (at 125.9055 190.4206 0)
       (effects (font (size 1.27 1.27)) (justify left) hide)
     )
@@
       (effects (font (size 1.27 1.27)) hide)
     )
+    (property "JLCPCB" "C49678" (id 4) (at 86.36 200.66 90)
+      (effects (font (size 1.27 1.27)) hide)
+    )
